File: PCB/AntSwitcher/AntSwitcher.sch (KiCad schematic (older format))
At the start: 33 parts, among them J1 Barrel_Jack, J2 TRX_UKW, J3 TRX2, J4 ANT1, J5 ANT2, K1 HF3-53, K2 HF3-53, K3 HF3-53, K4 HF3-53, Q1 Q_NMOS_GSD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

Commit message: HF-Layout Relays
Parts:
- D5, D6, D8, D9: symbol Device:D -> DiodeFlyback:D
Connections:
- net GNDREF: now also D5.1 (A), D6.1 (A), D8.1 (A), D9.1 (A); no longer D5.2 (A), D6.2 (A), D8.2 (A), D9.2 (A)
- net at K1.11, Q2.3 (D): now also D5.3 (K); no longer D5.1 (K)
- net at K3.11, Q3.3 (D): now also D8.3 (K); no longer D8.1 (K)
- net at K4.11, Q4.3 (D): now also D9.3 (K); no longer D9.1 (K)
- net at K2.11, Q1.3 (D): now also D6.3 (K); no longer D6.1 (K)
Changed lines of the file:
@@
 	8900 1350 8700 1350
-$Comp
-L Device:Q_NJFET_GSD Q4
-U 1 1 5ED155EF
-P 6650 4400
-F 0 "Q4" H 6854 4446 50  0000 L CNN
-F 1 "Q_NMOS_GSD" H 6854 4355 50  0000 L CNN
-F 2 "TO_SOT_Packages_SMD:SOT-23" H 6850 4500 50  0001 C CNN
-F 3 "~" H 6650 4400 50  0001 C CNN
-	1    6650 4400
-	1    0    0    -1
-$EndComp
 $Comp
 L power:GNDREF #PWR021
@@
 	8000 2700 8100 2700
 $Comp
-L Device:D D8
+L DiodeFlyback:D D8
 U 1 1 5EDD0315
 P 9150 1150
@@
 	8900 1000 9150 1000
 $Comp
-L Device:D D5
+L DiodeFlyback:D D5
 U 1 1 5EDD7DC0
 P 6050 1500
@@
 $EndComp
 $Comp
-L Device:D D9
-U 1 1 5EDD8BFF
-P 9150 2550
-F 0 "D9" V 9104 2630 50  0000 L CNN
-F 1 "D" V 9195 2630 50  0000 L CNN
-F 2 "TO_SOT_Packages_SMD:SOT-23" H 9150 2550 50  0001 C CNN
-F 3 "~" H 9150 2550 50  0001 C CNN
-	1    9150 2550
-	0    1    1    0
-$EndComp
-$Comp
 L power:GNDREF #PWR030
 U 1 1 5EDDA455
@@
 	1    0    0    -1
 $EndComp
-Wire Wire Line
-	9150 2400 9000 2400
-Wire Wire Line
-	9000 2400 9000 2700
 $Comp
 L power:GNDREF #PWR09
@@
 	6850 2950 7100 2950
 $Comp
-L Device:D D6
+L DiodeFlyback:D D6
 U 1 1 5EDF950F
 P 6150 2800
@@
 Wire Wire Line
 	9650 4200 9650 2400
-Wire Wire Line
-	9650 2400 9150 2400
-Connection ~ 9150 2400
 $Comp
 L Device:R R4
@@
 Wire Wire Line
 	6850 2650 6950 2650
+$Comp
+L Device:Q_NJFET_GSD Q4
+U 1 1 5ED155EF
+P 6650 4400
+F 0 "Q4" H 6854 4446 50  0000 L CNN
+F 1 "Q_NMOS_GSD" H 6854 4355 50  0000 L CNN
+F 2 "TO_SOT_Packages_SMD:SOT-23" H 6850 4500 50  0001 C CNN
+F 3 "~" H 6650 4400 50  0001 C CNN
+	1    6650 4400
+	1    0    0    -1
+$EndComp
+$Comp
+L DiodeFlyback:D D9
+U 1 1 5EDD8BFF
+P 9150 2550
+F 0 "D9" V 9104 2630 50  0000 L CNN
+F 1 "D" V 9195 2630 50  0000 L CNN
+F 2 "TO_SOT_Packages_SMD:SOT-23" H 9150 2550 50  0001 C CNN
+F 3 "~" H 9150 2550 50  0001 C CNN
+	1    9150 2550
+	0    1    1    0
+$EndComp
+Wire Wire Line
+	9000 2400 9150 2400
+Wire Wire Line
+	9150 2400 9650 2400
+Connection ~ 9150 2400
+Wire Wire Line
+	9000 2400 9000 2700
 $EndSCHEMATC

Commit message: Barrel Jack changed to SMD variant
Parts:
- J1: footprint Connectors:BARREL_JACK -> BarrelJackSMD:BarrelJackSMD
Changed lines of the file:
@@
 F 0 "J1" H 3907 6075 50  0000 C CNN
 F 1 "Barrel_Jack" H 3907 5984 50  0000 C CNN
-F 2 "Connectors:BARREL_JACK" H 3900 5710 50  0001 C CNN
+F 2 "BarrelJackSMD:BarrelJackSMD" H 3900 5710 50  0001 C CNN
 F 3 "~" H 3900 5710 50  0001 C CNN
 	1    3850 5750
